Commit message: URDF visualized successfuly in RVIZ

File: src/myrobot_sim/urdf/Trial_idk.urdf (robot description, URDF)
Before this commit: robot Trial_idk, 7 links, 6 joints
Joints:
- joint FR_Wheel_Joint: axis 0 0 1 -> 0 0 -1
- joint Pinion_Joint: axis 0 0 1 -> 0 0 -1
- joint RR_Wheel_Joint: axis 0 0 1 -> 0 0 -1

Commit message: hi gazebo trial

File: src/myrobot_sim/urdf/Trial_idk.urdf (robot description, URDF)
Before this commit: robot Trial_idk, 7 links, 6 joints
Links:
- link Arm: geometry collision mesh filename=file:///home/roaa/My_Workspace/install/myrobot_sim/share/my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; visual mesh filename=file:///home/roaa/My_Workspace/install/myrobot_sim/share/my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
- link FL_Wheel: geometry collision mesh filename=file:///home/roaa/My_Workspace/install/myrobot_sim/share/my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; visual mesh filename=file:///home/roaa/My_Workspace/install/myrobot_sim/share/my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
- link FR_Wheel: geometry collision mesh filename=file:///home/roaa/My_Workspace/install/myrobot_sim/share/my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; visual mesh filename=file:///home/roaa/My_Workspace/install/myrobot_sim/share/my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
- link Pinion: geometry collision mesh filename=file:///home/roaa/My_Workspace/install/myrobot_sim/share/my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; visual mesh filename=file:///home/roaa/My_Workspace/install/myrobot_sim/share/my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
- link RL_Wheel: geometry collision mesh filename=file:///home/roaa/My_Workspace/install/myrobot_sim/share/my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; visual mesh filename=file:///home/roaa/My_Workspace/install/myrobot_sim/share/my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
- link RR_Wheel: geometry collision mesh filename=file:///home/roaa/My_Workspace/install/myrobot_sim/share/my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; visual mesh filename=file:///home/roaa/My_Workspace/install/myrobot_sim/share/my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
- link base_link: geometry collision mesh filename=file:///home/roaa/My_Workspace/install/myrobot_sim/share/my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; visual mesh filename=file:///home/roaa/My_Workspace/install/myrobot_sim/share/my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

Commit message: Gazebo visualized initially

File: src/myrobot_sim/urdf/Trial_idk.urdf (robot description, URDF)
Before this commit: robot Trial_idk, 7 links, 6 joints
Links:
- link Arm: geometry collision mesh filename=file:///home/sara/design2_ws/install/myrobot_sim/share/myro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; visual mesh filename=file:///home/sara/design2_ws/install/myrobot_sim/share/myro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
- link FL_Wheel: geometry collision mesh filename=file:///home/sara/design2_ws/install/myrobot_sim/share/myro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; visual mesh filename=file:///home/sara/design2_ws/install/myrobot_sim/share/myro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
- link FR_Wheel: geometry collision mesh filename=file:///home/sara/design2_ws/install/myrobot_sim/share/myro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; visual mesh filename=file:///home/sara/design2_ws/install/myrobot_sim/share/myro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
- link Pinion: geometry collision mesh filename=file:///home/sara/design2_ws/install/myrobot_sim/share/myro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; visual mesh filename=file:///home/sara/design2_ws/install/myrobot_sim/share/myro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
- link RL_Wheel: geometry collision mesh filename=file:///home/sara/design2_ws/install/myrobot_sim/share/myro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; visual mesh filename=file:///home/sara/design2_ws/install/myrobot_sim/share/myro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
- link RR_Wheel: geometry collision mesh filename=file:///home/sara/design2_ws/install/myrobot_sim/share/myro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; visual mesh filename=file:///home/sara/design2_ws/install/myrobot_sim/share/myro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
- link base_link: geometry collision mesh filename=file:///home/sara/design2_ws/install/myrobot_sim/share/myro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; visual mesh filename=file:///home/sara/design2_ws/install/myrobot_sim/share/myro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

Commit message: Ultrasonic added and visualized with the IMU

File: src/myrobot_sim/urdf/Trial_idk.urdf (robot description, URDF)
Before this commit: robot Trial_idk, 7 links, 6 joints
Links:
- added link imu_link, mass 0.05; collision box size=0.02 0.02 0.01; visual box size=0.02 0.02 0.01
- added link ultrasonic_link, mass 0.1; collision cylinder length=0.05 radius=0.03; visual cylinder length=0.05 radius=0.03
- link Arm: geometry collision mesh filename=file:///home/roaa/My_Workspace/install/myrobot_sim/share/my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; visual mesh filename=file:///home/roaa/My_Workspace/install/myrobot_sim/share/my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
- link FL_Wheel: geometry collision mesh filename=file:///home/roaa/My_Workspace/install/myrobot_sim/share/my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; visual mesh filename=file:///home/roaa/My_Workspace/install/myrobot_sim/share/my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
- link FR_Wheel: geometry collision mesh filename=file:///home/roaa/My_Workspace/install/myrobot_sim/share/my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; visual mesh filename=file:///home/roaa/My_Workspace/install/myrobot_sim/share/my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
- link Pinion: geometry collision mesh filename=file:///home/roaa/My_Workspace/install/myrobot_sim/share/my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; visual mesh filename=file:///home/roaa/My_Workspace/install/myrobot_sim/share/my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
- link RL_Wheel: geometry collision mesh filename=file:///home/roaa/My_Workspace/install/myrobot_sim/share/my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; visual mesh filename=file:///home/roaa/My_Workspace/install/myrobot_sim/share/my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
- link RR_Wheel: geometry collision mesh filename=file:///home/roaa/My_Workspace/install/myrobot_sim/share/my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; visual mesh filename=file:///home/roaa/My_Workspace/install/myrobot_sim/share/my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
- link base_link: geometry collision mesh filename=file:///home/roaa/My_Workspace/install/myrobot_sim/share/my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; visual mesh filename=file:///home/roaa/My_Workspace/install/myrobot_sim/share/my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
Joints:
- added joint imu_joint: type fixed, parent base_link, child imu_link, origin xyz=0 0 0.05 rpy=0 0 0
- added joint ultrasonic_joint: type fixed, parent base_link, child ultrasonic_link, origin xyz=0.15 0 0.07 rpy=0 0 0

Commit message: 2 labs done but with some errors yet to be handeled

File: src/myrobot_sim/urdf/Trial_idk.urdf (robot description, URDF)
Before this commit: robot Trial_idk, 9 links, 8 joints
Joints:
- joint Arm_Joint: mimic joint=Pinion_Joint multiplier=2.5 offset=0 -> (none)

Commit message: Static obstacle avoidance state machine works, needs further refinment

File: src/myrobot_sim/urdf/Trial_idk.urdf (robot description, URDF)
Before this commit: robot Trial_idk, 9 links, 8 joints
Joints:
- joint ultrasonic_joint: origin xyz=0.15 0 0.07 rpy=0 0 0 -> xyz=0.15 0 -0.1 rpy=0 0 0

Commit message: Obstacle avoidance both static and dynamic done

File: src/myrobot_sim/urdf/Trial_idk.urdf (robot description, URDF)
Before this commit: robot Trial_idk, 9 links, 8 joints
Links:
- removed link ultrasonic_link
- added link ultrasonic_center_link, mass 0.1; collision cylinder length=0.05 radius=0.03; visual cylinder length=0.05 radius=0.03
- added link ultrasonic_left_link, mass 0.1; collision cylinder length=0.05 radius=0.03; visual cylinder length=0.05 radius=0.03
- added link ultrasonic_right_link, mass 0.1; collision cylinder length=0.05 radius=0.03; visual cylinder length=0.05 radius=0.03
Joints:
- removed joint ultrasonic_joint
- added joint ultrasonic_center_joint: type fixed, parent base_link, child ultrasonic_center_link, origin xyz=0.15 0 -0.1 rpy=0 0 0
- added joint ultrasonic_left_joint: type fixed, parent base_link, child ultrasonic_left_link, origin xyz=0.128 0.115 -0.1 rpy=0 0 0.5236
- added joint ultrasonic_right_joint: type fixed, parent base_link, child ultrasonic_right_link, origin xyz=0.128 -0.115 -0.1 rpy=0 0 -0.5236

Commit message: Logic done fadel tafseela fl avoidance w el environment

File: src/myrobot_sim/urdf/Trial_idk.urdf (robot description, URDF)
Before this commit: robot Trial_idk, 11 links, 10 joints
Joints:
- joint Arm_Joint: limit lower=0 upper=3.14 effort=10 velocity=1 -> lower=-3.14 upper=3.14 effort=10 velocity=1
